File: kicad/zillo-mini-devkit/_autosave-zillo-mini-devkit.sch (KiCad schematic (older format))
At the start: 9 parts, among them J1 Conn_01x19, J2 Conn_01x19, J3 Conn_01x08

Commit message: kicad
Connections:
- net GND: now also J1.7 (Pin_7)
- net LEDMATRIX: now also J2.11 (Pin_11)
Changed lines of the file:
@@
 GND
 $Comp
-L power:GND #PWR?
+L power:GND #PWR0108
 U 1 1 5DE04BD4
 P 5350 1650
-F 0 "#PWR?" H 5350 1400 50  0001 C CNN
+F 0 "#PWR0108" H 5350 1400 50  0001 C CNN
 F 1 "GND" H 5355 1477 50  0000 C CNN
 F 2 "" H 5350 1650 50  0001 C CNN
@@
 Wire Wire Line
 	5350 1550 5450 1550
+Text GLabel 5450 1850 2    50   Output ~ 0
+LEDMATRIX
+Wire Wire Line
+	5050 1850 5450 1850
+Text GLabel 3500 2250 0    50   UnSpc ~ 0
+GND
+$Comp
+L power:GND #PWR0109
+U 1 1 5DE1D0B1
+P 3600 2150
+F 0 "#PWR0109" H 3600 1900 50  0001 C CNN
+F 1 "GND" H 3605 1977 50  0000 C CNN
+F 2 "" H 3600 2150 50  0001 C CNN
+F 3 "" H 3600 2150 50  0001 C CNN
+	1    3600 2150
+	-1   0    0    1
+$EndComp
+Wire Wire Line
+	3750 2250 3600 2250
+Wire Wire Line
+	3600 2150 3600 2250
+Connection ~ 3600 2250
+Wire Wire Line
+	3600 2250 3500 2250
 $EndSCHEMATC
